Commit message: ros2_control_launch_fixed

File: rom2109_description/urdf/urdf.urdf (robot description, URDF)
Before this commit: robot rom2109, 10 links, 9 joints
Links:
- link base_link: geometry collision mesh filename=/home/zyme/.gazebo/models/rom2109_tall/meshes/tall/base_lin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; visual mesh filename=/home/zyme/.gazebo/models/rom2109_tall/meshes/tall/base_lin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
- link camera: geometry collision mesh filename=/home/zyme/.gazebo/models/rom2109_tall/meshes/tall/camera.S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; visual mesh filename=/home/zyme/.gazebo/models/rom2109_tall/meshes/tall/camera.S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
- link left_wheel: geometry collision mesh filename=/home/zyme/.gazebo/models/rom2109_tall/meshes/tall/left_whe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; visual mesh filename=/home/zyme/.gazebo/models/rom2109_tall/meshes/tall/left_whe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
- link lidar: geometry collision mesh filename=/home/zyme/.gazebo/models/rom2109_tall/meshes/tall/lidar.STL; visual mesh filename=/home/zyme/.gazebo/models/rom2109_tall/meshes/tall/lidar.STL
- link plate1: geometry collision mesh filename=/home/zyme/.gazebo/models/rom2109_tall/meshes/tall/plate1.S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; visual mesh filename=/home/zyme/.gazebo/models/rom2109_tall/meshes/tall/plate1.S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
- link plate2: geometry collision mesh filename=/home/zyme/.gazebo/models/rom2109_tall/meshes/tall/plate2.S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; visual mesh filename=/home/zyme/.gazebo/models/rom2109_tall/meshes/tall/plate2.S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
- link plate3: geometry collision mesh filename=/home/zyme/.gazebo/models/rom2109_tall/meshes/tall/plate3.S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; visual mesh filename=/home/zyme/.gazebo/models/rom2109_tall/meshes/tall/plate3.S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
- link right_wheel: geometry collision mesh filename=/home/zyme/.gazebo/models/rom2109_tall/meshes/tall/right_wh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; visual mesh filename=/home/zyme/.gazebo/models/rom2109_tall/meshes/tall/right_wh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

Commit message: I added the path_replacer in ::rom2109_description/urdf/ (that replace the org file path to our system file path

File: rom2109_description/urdf/urdf.urdf (robot description, URDF)
Before this commit: robot rom2109, 10 links, 9 joints
Links:
- link base_link: geometry collision mesh filename=/home/rom/.gazebo/models/rom2109_tall/meshes/tall/base_link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; visual mesh filename=/home/rom/.gazebo/models/rom2109_tall/meshes/tall/base_link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
- link camera: geometry collision mesh filename=/home/rom/.gazebo/models/rom2109_tall/meshes/tall/camera.STL; visual mesh filename=/home/rom/.gazebo/models/rom2109_tall/meshes/tall/camera.STL
- link left_wheel: geometry collision mesh filename=/home/rom/.gazebo/models/rom2109_tall/meshes/tall/left_whee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; visual mesh filename=/home/rom/.gazebo/models/rom2109_tall/meshes/tall/left_whee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
- link lidar: geometry collision mesh filename=/home/rom/.gazebo/models/rom2109_tall/meshes/tall/lidar.STL; visual mesh filename=/home/rom/.gazebo/models/rom2109_tall/meshes/tall/lidar.STL
- link plate1: geometry collision mesh filename=/home/rom/.gazebo/models/rom2109_tall/meshes/tall/plate1.STL; visual mesh filename=/home/rom/.gazebo/models/rom2109_tall/meshes/tall/plate1.STL
- link plate2: geometry collision mesh filename=/home/rom/.gazebo/models/rom2109_tall/meshes/tall/plate2.STL; visual mesh filename=/home/rom/.gazebo/models/rom2109_tall/meshes/tall/plate2.STL
- link plate3: geometry collision mesh filename=/home/rom/.gazebo/models/rom2109_tall/meshes/tall/plate3.STL; visual mesh filename=/home/rom/.gazebo/models/rom2109_tall/meshes/tall/plate3.STL
- link right_wheel: geometry collision mesh filename=/home/rom/.gazebo/models/rom2109_tall/meshes/tall/right_whe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; visual mesh filename=/home/rom/.gazebo/models/rom2109_tall/meshes/tall/right_whe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

Commit message: mapping OK

File: rom2109_description/urdf/urdf.urdf (robot description, URDF)
Before this commit: robot rom2109, 10 links, 9 joints
Links:
- link base_link: geometry collision mesh filename=/home/mr_robot/.gazebo/models/rom2109_tall/meshes/tall/base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; visual mesh filename=/home/mr_robot/.gazebo/models/rom2109_tall/meshes/tall/base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
- link camera: geometry collision mesh filename=/home/mr_robot/.gazebo/models/rom2109_tall/meshes/tall/came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; visual mesh filename=/home/mr_robot/.gazebo/models/rom2109_tall/meshes/tall/came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
- link left_wheel: geometry collision mesh filename=/home/mr_robot/.gazebo/models/rom2109_tall/meshes/tall/left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; visual mesh filename=/home/mr_robot/.gazebo/models/rom2109_tall/meshes/tall/left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
- link lidar: geometry collision mesh filename=/home/mr_robot/.gazebo/models/rom2109_tall/meshes/tall/lida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; visual mesh filename=/home/mr_robot/.gazebo/models/rom2109_tall/meshes/tall/lida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
- link plate1: geometry collision mesh filename=/home/mr_robot/.gazebo/models/rom2109_tall/meshes/tall/plat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; visual mesh filename=/home/mr_robot/.gazebo/models/rom2109_tall/meshes/tall/plat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
- link plate2: geometry collision mesh filename=/home/mr_robot/.gazebo/models/rom2109_tall/meshes/tall/plat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; visual mesh filename=/home/mr_robot/.gazebo/models/rom2109_tall/meshes/tall/plat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
- link plate3: geometry collision mesh filename=/home/mr_robot/.gazebo/models/rom2109_tall/meshes/tall/plat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; visual mesh filename=/home/mr_robot/.gazebo/models/rom2109_tall/meshes/tall/plat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
- link right_wheel: geometry collision mesh filename=/home/mr_robot/.gazebo/models/rom2109_tall/meshes/tall/righ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; visual mesh filename=/home/mr_robot/.gazebo/models/rom2109_tall/meshes/tall/righ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

Commit message: collision monitor add

File: rom2109_description/urdf/urdf.urdf (robot description, URDF)
Before this commit: robot rom2109, 10 links, 9 joints
Links:
- link base_link: geometry collision mesh filename=/home/catto/.gazebo/models/rom2109_tall/meshes/tall/base_li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; visual mesh filename=/home/catto/.gazebo/models/rom2109_tall/meshes/tall/base_li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
- link camera: geometry collision mesh filename=/home/catto/.gazebo/models/rom2109_tall/meshes/tall/camera.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; visual mesh filename=/home/catto/.gazebo/models/rom2109_tall/meshes/tall/camera.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
- link left_wheel: geometry collision mesh filename=/home/catto/.gazebo/models/rom2109_tall/meshes/tall/left_wh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; visual mesh filename=/home/catto/.gazebo/models/rom2109_tall/meshes/tall/left_wh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
- link lidar: geometry collision mesh filename=/home/catto/.gazebo/models/rom2109_tall/meshes/tall/lidar.S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; visual mesh filename=/home/catto/.gazebo/models/rom2109_tall/meshes/tall/lidar.S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
- link plate1: geometry collision mesh filename=/home/catto/.gazebo/models/rom2109_tall/meshes/tall/plate1.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; visual mesh filename=/home/catto/.gazebo/models/rom2109_tall/meshes/tall/plate1.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
- link plate2: geometry collision mesh filename=/home/catto/.gazebo/models/rom2109_tall/meshes/tall/plate2.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; visual mesh filename=/home/catto/.gazebo/models/rom2109_tall/meshes/tall/plate2.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
- link plate3: geometry collision mesh filename=/home/catto/.gazebo/models/rom2109_tall/meshes/tall/plate3.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; visual mesh filename=/home/catto/.gazebo/models/rom2109_tall/meshes/tall/plate3.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
- link right_wheel: geometry collision mesh filename=/home/catto/.gazebo/models/rom2109_tall/meshes/tall/right_w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; visual mesh filename=/home/catto/.gazebo/models/rom2109_tall/meshes/tall/right_w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

Commit message: course ros2_control

File: rom2109_description/urdf/urdf.urdf (robot description, URDF)
Before this commit: robot rom2109, 10 links, 9 joints
Links:
- link base_link: geometry collision mesh filename=package://rom2109_description/meshes/tall/base_link.STL; visual mesh filename=package://rom2109_description/meshes/tall/base_link.STL
- link camera: geometry collision mesh filename=package://rom2109_description/meshes/tall/camera.STL; visual mesh filename=package://rom2109_description/meshes/tall/camera.STL
- link left_wheel: geometry collision mesh filename=package://rom2109_description/meshes/tall/left_wheel.STL; visual mesh filename=package://rom2109_description/meshes/tall/left_wheel.STL
- link lidar: geometry collision mesh filename=package://rom2109_description/meshes/tall/lidar.STL; visual mesh filename=package://rom2109_description/meshes/tall/lidar.STL
- link plate1: geometry collision mesh filename=package://rom2109_description/meshes/tall/plate1.STL; visual mesh filename=package://rom2109_description/meshes/tall/plate1.STL
- link plate2: geometry collision mesh filename=package://rom2109_description/meshes/tall/plate2.STL; visual mesh filename=package://rom2109_description/meshes/tall/plate2.STL
- link plate3: geometry collision mesh filename=package://rom2109_description/meshes/tall/plate3.STL; visual mesh filename=package://rom2109_description/meshes/tall/plate3.STL
- link right_wheel: geometry collision mesh filename=package://rom2109_description/meshes/tall/right_wheel.STL; visual mesh filename=package://rom2109_description/meshes/tall/right_wheel.STL
