Commit message: ekf unstable

File: rom2109_description/urdf/rom2109_core.xacro (robot description, xacro)
@@ -418,4 +418,10 @@
       xyz="0 0 0" />
   </joint>
+    <link name="imu_link"/>
+    <joint name="imu_joint" type="fixed">
+      <parent link="base_link"/>
+      <child link="imu_link"/>
+      <origin rpy="0 0 0" xyz="0 0 0"/>
+    </joint>
   <!-- Colour -->
   <gazebo reference="base_link">

File: rom2109_description/urdf/sim_ros2_control.xacro (robot description, xacro)
@@ -35,3 +35,23 @@
         </plugin>
     </gazebo>
+    <gazebo reference="imu_link">
+        <gravity>true</gravity>
+        <sensor name="imu_sensor" type="imu">
+            <always_on>true</always_on>
+            <update_rate>20</update_rate>
+            <visualize>true</visualize>
+            <topic>/imu</topic>
+            <plugin filename="libgazebo_ros_imu_sensor.so" name="imu_plugin">
+                <topicName>imu</topicName>
+                <bodyName>imu_link</bodyName>
+                <updateRateHZ>10.0</updateRateHZ>
+                <gaussianNoise>0.0</gaussianNoise>
+                <xyzOffset>0 0 0</xyzOffset>
+                <rpyOffset>0 0 0</rpyOffset>
+                <frameName>imu_link</frameName>
+                <initialOrientationAsReference>false</initialOrientationAsReference>
+            </plugin>
+            <pose>0 0 0 0 0 0</pose>
+        </sensor>
+    </gazebo>
 </robot>

File: rom2109_description/urdf/yoururdf.urdf (robot description, URDF)
Before this commit: robot rom2109, 10 links, 9 joints
Links:
- added link imu_link
Joints:
- added joint imu_joint: type fixed, parent base_link, child imu_link, origin xyz=0 0 0 rpy=0 0 0
