Commit message: ros2 control ready

File: rom2109_description/urdf/robot_sim_ros2_control.urdf.xacro (robot description, xacro)
@@ -2,7 +2,7 @@
 <robot xmlns:xacro="http://www.ros.org/wiki/xacro"  name="rom2109">
     <xacro:include filename="rom2109_core.xacro" />
+    <xacro:include filename="sim_ros2_control.xacro" />
     <xacro:include filename="lidar.xacro" />
     <!-- <xacro:include filename="hw_ros2_control.xacro" />  -->
-    <xacro:include filename="ros2_control.xacro" />
     <!-- <xacro:include filename="gazebo_control.xacro" /> -->
     <xacro:include filename="camera.xacro" />

File: rom2109_description/urdf/yoururdf.urdf (robot description, URDF)
Before this commit: robot rom2109, 10 links, 9 joints
Links:
- link base_link: geometry collision mesh filename=/home/mr_robot/ros2/developer_ws/src/rom2109_simulation/rom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; visual mesh filename=/home/mr_robot/ros2/developer_ws/src/rom2109_simulation/rom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
- link camera: geometry collision mesh filename=/home/mr_robot/ros2/developer_ws/src/rom2109_simulation/rom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; visual mesh filename=/home/mr_robot/ros2/developer_ws/src/rom2109_simulation/rom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
- link left_wheel: geometry collision mesh filename=/home/mr_robot/ros2/developer_ws/src/rom2109_simulation/rom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; visual mesh filename=/home/mr_robot/ros2/developer_ws/src/rom2109_simulation/rom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
- link lidar: geometry collision mesh filename=/home/mr_robot/ros2/developer_ws/src/rom2109_simulation/rom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; visual mesh filename=/home/mr_robot/ros2/developer_ws/src/rom2109_simulation/rom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
- link plate1: geometry collision mesh filename=/home/mr_robot/ros2/developer_ws/src/rom2109_simulation/rom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; visual mesh filename=/home/mr_robot/ros2/developer_ws/src/rom2109_simulation/rom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
- link plate2: geometry collision mesh filename=/home/mr_robot/ros2/developer_ws/src/rom2109_simulation/rom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; visual mesh filename=/home/mr_robot/ros2/developer_ws/src/rom2109_simulation/rom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
- link plate3: geometry collision mesh filename=/home/mr_robot/ros2/developer_ws/src/rom2109_simulation/rom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; visual mesh filename=/home/mr_robot/ros2/developer_ws/src/rom2109_simulation/rom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
- link right_wheel: geometry collision mesh filename=/home/mr_robot/ros2/developer_ws/src/rom2109_simulation/rom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; visual mesh filename=/home/mr_robot/ros2/developer_ws/src/rom2109_simulation/rom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

Commit message: spawning_gazebo_error

File: rom2109_description/urdf/robot_sim_ros2_control.urdf.xacro (robot description, xacro)
@@ -2,5 +2,5 @@
 <robot xmlns:xacro="http://www.ros.org/wiki/xacro"  name="rom2109">
     <xacro:include filename="rom2109_core.xacro" />
-    <xacro:include filename="sim_ros2_control.xacro" />
+    <!-- <xacro:include filename="sim_ros2_control.xacro" />  -->
     <xacro:include filename="lidar.xacro" />
     <!-- <xacro:include filename="hw_ros2_control.xacro" />  -->

File: rom2109_description/urdf/rom2109_core.xacro (robot description, xacro)
@@ -1,4 +1,4 @@
 <?xml version="1.0"?>
-<robot xmlns:xacro="http://www.ros.org/wiki/xacro">
+<robot xmlns:xacro="http://www.ros.org/wiki/xacro" name="rom2109_tall_ros">
     <link name="base_footprint"></link>
     <joint name="base_footprint_joint" type="fixed">

File: rom2109_description/urdf/sim_ros2_control.xacro (robot description, xacro)
@@ -24,6 +24,6 @@
     <gazebo>
         <plugin name="gazebo_ros2_control" filename="libgazebo_ros2_control.so">
-            <robot_param>robot_description</robot_param>
-            <robot_param_node>robot_state_publisher</robot_param_node>
+            <!-- <robot_param>robot_description</robot_param>
+            <robot_param_node>robot_state_publisher</robot_param_node> -->
             <parameters>$(find rom2109_description)/config/my_controllers.yaml</parameters>
             <!-- Output -->

File: rom2109_description/urdf/yoururdf.urdf (robot description, URDF)
Before this commit: robot rom2109, 11 links, 10 joints
Links:
- link base_link: geometry collision mesh filename=/home/zyme/.gazebo/models/rom2109_description/rom2109_descr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; visual mesh filename=/home/zyme/.gazebo/models/rom2109_description/rom2109_descr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
- link camera: geometry collision mesh filename=/home/zyme/.gazebo/models/rom2109_description/rom2109_descr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; visual mesh filename=/home/zyme/.gazebo/models/rom2109_description/rom2109_descr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
- link left_wheel: geometry collision mesh filename=/home/zyme/.gazebo/models/rom2109_description/rom2109_descr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; visual mesh filename=/home/zyme/.gazebo/models/rom2109_description/rom2109_descr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
- link lidar: geometry collision mesh filename=/home/zyme/.gazebo/models/rom2109_description/rom2109_descr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; visual mesh filename=/home/zyme/.gazebo/models/rom2109_description/rom2109_descr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
- link plate1: geometry collision mesh filename=/home/zyme/.gazebo/models/rom2109_description/rom2109_descr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; visual mesh filename=/home/zyme/.gazebo/models/rom2109_description/rom2109_descr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
- link plate2: geometry collision mesh filename=/home/zyme/.gazebo/models/rom2109_description/rom2109_descr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; visual mesh filename=/home/zyme/.gazebo/models/rom2109_description/rom2109_descr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
- link plate3: geometry collision mesh filename=/home/zyme/.gazebo/models/rom2109_description/rom2109_descr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; visual mesh filename=/home/zyme/.gazebo/models/rom2109_description/rom2109_descr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
- link right_wheel: geometry collision mesh filename=/home/zyme/.gazebo/models/rom2109_description/rom2109_descr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; visual mesh filename=/home/zyme/.gazebo/models/rom2109_description/rom2109_descr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
