Commit message: shell update

File: rom2109_description/urdf/yoururdf.urdf (robot description, URDF)
Before this commit: robot rom2109, 11 links, 10 joints
Links:
- link base_link: geometry collision mesh filename=/home/mr_robot/.gazebo/models/rom2109_description/rom2109_d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; visual mesh filename=/home/mr_robot/.gazebo/models/rom2109_description/rom2109_d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
- link camera: geometry collision mesh filename=/home/mr_robot/.gazebo/models/rom2109_description/rom2109_d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; visual mesh filename=/home/mr_robot/.gazebo/models/rom2109_description/rom2109_d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
- link left_wheel: geometry collision mesh filename=/home/mr_robot/.gazebo/models/rom2109_description/rom2109_d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; visual mesh filename=/home/mr_robot/.gazebo/models/rom2109_description/rom2109_d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
- link lidar: geometry collision mesh filename=/home/mr_robot/.gazebo/models/rom2109_description/rom2109_d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; visual mesh filename=/home/mr_robot/.gazebo/models/rom2109_description/rom2109_d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
- link plate1: geometry collision mesh filename=/home/mr_robot/.gazebo/models/rom2109_description/rom2109_d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; visual mesh filename=/home/mr_robot/.gazebo/models/rom2109_description/rom2109_d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
- link plate2: geometry collision mesh filename=/home/mr_robot/.gazebo/models/rom2109_description/rom2109_d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; visual mesh filename=/home/mr_robot/.gazebo/models/rom2109_description/rom2109_d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
- link plate3: geometry collision mesh filename=/home/mr_robot/.gazebo/models/rom2109_description/rom2109_d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; visual mesh filename=/home/mr_robot/.gazebo/models/rom2109_description/rom2109_d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
- link right_wheel: geometry collision mesh filename=/home/mr_robot/.gazebo/models/rom2109_description/rom2109_d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; visual mesh filename=/home/mr_robot/.gazebo/models/rom2109_description/rom2109_d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

Commit message: spawn_with_file::fine

File: rom2109_description/urdf/yoururdf.urdf (robot description, URDF)
Before this commit: robot rom2109, 11 links, 10 joints
Links:
- link base_link: geometry collision mesh filename=/home/zyme/ros_ws/rom2109_sim/src/rom2109_simulation/rom210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; visual mesh filename=/home/zyme/ros_ws/rom2109_sim/src/rom2109_simulation/rom210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
- link camera: geometry collision mesh filename=/home/zyme/ros_ws/rom2109_sim/src/rom2109_simulation/rom210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; visual mesh filename=/home/zyme/ros_ws/rom2109_sim/src/rom2109_simulation/rom210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
- link left_wheel: geometry collision mesh filename=/home/zyme/ros_ws/rom2109_sim/src/rom2109_simulation/rom210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; visual mesh filename=/home/zyme/ros_ws/rom2109_sim/src/rom2109_simulation/rom210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
- link lidar: geometry collision mesh filename=/home/zyme/ros_ws/rom2109_sim/src/rom2109_simulation/rom210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; visual mesh filename=/home/zyme/ros_ws/rom2109_sim/src/rom2109_simulation/rom210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
- link plate1: geometry collision mesh filename=/home/zyme/ros_ws/rom2109_sim/src/rom2109_simulation/rom210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; visual mesh filename=/home/zyme/ros_ws/rom2109_sim/src/rom2109_simulation/rom210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
- link plate2: geometry collision mesh filename=/home/zyme/ros_ws/rom2109_sim/src/rom2109_simulation/rom210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; visual mesh filename=/home/zyme/ros_ws/rom2109_sim/src/rom2109_simulation/rom210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
- link plate3: geometry collision mesh filename=/home/zyme/ros_ws/rom2109_sim/src/rom2109_simulation/rom210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; visual mesh filename=/home/zyme/ros_ws/rom2109_sim/src/rom2109_simulation/rom210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
- link right_wheel: geometry collision mesh filename=/home/zyme/ros_ws/rom2109_sim/src/rom2109_simulation/rom210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; visual mesh filename=/home/zyme/ros_ws/rom2109_sim/src/rom2109_simulation/rom210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
